File: shvc/sdnes.kicad_pcb (KiCad board)
At the start: 2 copper layers, 17.5 x 23.4 mm, 5 parts, among them J1 500901-0801

Commit message: Fix silkscreen
Other:
- board text added: "SDNES SHVC github.com/ going-digital/ sdnes"
- board text removed: "SD mod for FTM-NES- Main-01 by Cathedrow"
- board text removed: "SD mod for FTM-SHVC- Main-01 by Cathedrow"
Changed lines of the file:
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@@
   (general
     (thickness 0.8)
-    (drawings 12)
+    (drawings 10)
     (tracks 81)
     (zones 0)
@@
     (34 B.Paste user hide)
     (35 F.Paste user hide)
-    (36 B.SilkS user hide)
-    (37 F.SilkS user hide)
+    (36 B.SilkS user)
+    (37 F.SilkS user)
     (38 B.Mask user)
     (39 F.Mask user hide)
@@
       (drillshape 0)
       (scaleselection 1)
-      (outputdirectory "./"))
+      (outputdirectory "fabrication/"))
   )
   (net 0 "")
@@
       (effects (font (size 1 1) (thickness 0.15)))
     )
-    (fp_text value "Red LED" (at -3.01 0 90) (layer F.Fab)
+    (fp_text value "Red LED" (at -0.092 1.522 90) (layer F.Fab)
       (effects (font (size 1 1) (thickness 0.15)))
     )
@@
     )
   )
-  (gr_text "SD mod for\nFTM-SHVC-\nMain-01\nby\nCathedrow" (at 149.352 104.14) (layer B.SilkS)
-    (effects (font (size 1.5 1.5) (thickness 0.3)) (justify mirror))
-  )
-  (gr_text "SD mod for\nFTM-NES-\nMain-01\nby\nCathedrow" (at 168.656 102.108) (layer B.SilkS)
-    (effects (font (size 1.5 1.5) (thickness 0.3)) (justify mirror))
-  )
-  (gr_text "Fit Molex\n500901" (at 166.624 102.616 90) (layer F.SilkS)
-    (effects (font (size 1.5 1.5) (thickness 0.3)))
+  (gr_text "SDNES SHVC\ngithub.com/\ngoing-digital/\nsdnes" (at 149 105) (layer B.SilkS)
+    (effects (font (size 1.5 1.3) (thickness 0.3)) (justify mirror))
   )
   (gr_text "Fit Molex\n500901" (at 149.352 106.426) (layer F.SilkS)
